Commit message: Added depth camera support

File: urdf/robot.urdf (robot description, URDF)
Before this commit: robot diff_drive_robot, 7 links, 6 joints
Links:
- added link camera_frame; collision box size=0.025 0.09 0.025; visual box size=0.025 0.09 0.025
Joints:
- added joint camera_joint: type fixed, parent chassis, child camera_frame, origin xyz=0.3 0 0.075 rpy=0 0 0

Commit message: Added support for rtabmap

File: urdf/robot.urdf (robot description, URDF)
Before this commit: robot diff_drive_robot, 8 links, 7 joints
Links:
- added link camera_optical_frame
Joints:
- added joint camera_optical_joint: type fixed, parent camera_frame, child camera_optical_frame, origin xyz=0 0 0 rpy=-1.57079632679 0 -1.57079632679
